File: electropneu/electropneu.kicad_sch (KiCad schematic)
At the start: 25 parts, among them J1 Barrel_Jack_Switch, J2 PWM_OUT_MOTOR, J3 12V_OUT_MOTOR, J4 PWM_OUT_VALVE, J5 12V_OUT_VALVE, J6 12V Terminal, Q1 LM7805, SW1 SW_SPDT, SW2 SW_SPDT

Commit message: Update README and schematic for pneumatic control board; add control mode logic and LED indicators in firmware
Other:
- company: YEA+ALFRESI -> aldrick-t
- title: Common Gripper Control Board Schematic -> Pneumatic Control Board Schematic
Changed lines of the file:
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@@
 	(paper "A4")
 	(title_block
-		(title "Common Gripper Control Board Schematic")
-		(date "2025-10-31")
-		(rev "R4")
-		(company "YEA+ALFRESI")
-		(comment 1 "Schematic by: Aldrick T")
+		(title "Pneumatic Control Board Schematic")
+		(date "2026-09-15")
+		(rev "R5")
+		(company "aldrick-t")
+		(comment 1 "Schematic by: Aldrick Tadeo")
 	)
 	(junction
